File: hardware/src/dpx_faded/dpx_faded.kicad_pcb (KiCad board)
At the start: 4 copper layers, 185.1 x 165 mm, 6 parts, among them J1 Conn_01x08_Pin, J2 Conn_01x08_Pin

Commit message: so much source and so much datasheet
lots of fader drama
gonna fork the design and reduce featureset, add x32 faders due to availa
basically make a FADE_4 clone first because well - that whole thing has turned into the mystery project
Parts:
- added C1: 4.7 uF, Capacitor_SMD:C_0805_2012Metric_Pad1.18x1.45mm_HandSolder, F.Cu at (-25.2, -66.2)
- added C10: 4.7 uF, Capacitor_SMD:C_0805_2012Metric_Pad1.18x1.45mm_HandSolder, F.Cu at (-25.2, -57.2)
- added C11: 100 uF, Capacitor_SMD:C_0603_1608Metric_Pad1.08x0.95mm_HandSolder, F.Cu at (-7.31, -53.8)
- added C12: 100 uF, Capacitor_SMD:C_0603_1608Metric_Pad1.08x0.95mm_HandSolder, F.Cu at (-7.31, -51.3)
- added C13: .1 uF, Capacitor_SMD:C_0805_2012Metric_Pad1.18x1.45mm_HandSolder, F.Cu at (-25.2, -54.2)
- added C14: 10uF, Capacitor_SMD:CP_Elec_5x5.8, F.Cu at (-18.3, -64.3)
- added C15: 10uF, Capacitor_SMD:C_0805_2012Metric_Pad1.18x1.45mm_HandSolder, F.Cu at (-25.2, -51.2)
- added C16: 10uF, Capacitor_SMD:CP_Elec_5x5.8, F.Cu at (-18.3, -57.5)
- added C17: 1 uF, Capacitor_SMD:C_0603_1608Metric_Pad1.08x0.95mm_HandSolder, F.Cu at (-7.31, -48.8)
- added C18: 1 uF, Capacitor_SMD:C_0603_1608Metric_Pad1.08x0.95mm_HandSolder, F.Cu at (-7.31, -46.3)
- added C19: 1 uF, Capacitor_SMD:C_0603_1608Metric_Pad1.08x0.95mm_HandSolder, F.Cu at (-2.96, -56.4)
- added C2: 100 uF, Capacitor_SMD:C_0603_1608Metric_Pad1.08x0.95mm_HandSolder, F.Cu at (-11.7, -56.4)
- added C3: 100 uF, Capacitor_SMD:C_0603_1608Metric_Pad1.08x0.95mm_HandSolder, F.Cu at (-11.7, -53.8)
- added C4: 4.7 uF, Capacitor_SMD:C_0805_2012Metric_Pad1.18x1.45mm_HandSolder, F.Cu at (-25.2, -63.2)
- added C5: 100 uF, Capacitor_SMD:C_0603_1608Metric_Pad1.08x0.95mm_HandSolder, F.Cu at (-11.7, -51.3)
- added C6: 100 uF, Capacitor_SMD:C_0603_1608Metric_Pad1.08x0.95mm_HandSolder, F.Cu at (-11.7, -48.8)
- added C7: 4.7 uF, Capacitor_SMD:C_0805_2012Metric_Pad1.18x1.45mm_HandSolder, F.Cu at (-25.2, -60.2)
- added C8: 100 uF, Capacitor_SMD:C_0603_1608Metric_Pad1.08x0.95mm_HandSolder, F.Cu at (-11.7, -46.3)
- added C9: 100 uF, Capacitor_SMD:C_0603_1608Metric_Pad1.08x0.95mm_HandSolder, F.Cu at (-7.31, -56.4)
- added D1: MBRA130LT3G, Diode_SMD:D_SMA, F.Cu at (8.25, -54.6)
- added D2: VBUS, DPX_LED:LED_0805_2012Metric_Pad1.15x1.40mm_HandSolder, F.Cu at (1.81, -66.2)
- added FB1: 220h 110mHz, DPX_USB:FERRITE_0603, F.Cu at (6.19, -35.2)
- added H1: MountingHole_Pad_MP, MountingHole:MountingHole_2.2mm_M2_ISO7380_Pad_TopBottom, F.Cu at (-30.1, -65.2)
- added H2: MountingHole_Pad_MP, MountingHole:MountingHole_2.2mm_M2_ISO7380_Pad_TopBottom, F.Cu at (-30.1, -60.2)
- added H3: MountingHole_Pad_MP, MountingHole:MountingHole_2.2mm_M2_ISO7380_Pad_TopBottom, F.Cu at (-30.1, -55.1)
- added H4: MountingHole_Pad_MP, MountingHole:MountingHole_2.2mm_M2_ISO7380_Pad_TopBottom, F.Cu at (-30.1, -50.1)
- added J3: motor.3, Connector_JST:JST_PH_B2B-PH-SM4-TB_1x02-1MP_P2.00mm_Vertical, F.Cu at (-43.0, -43.4)
- added J4: motor.4, Connector_JST:JST_PH_B2B-PH-SM4-TB_1x02-1MP_P2.00mm_Vertical, F.Cu at (-43.0, -33.8)
- added J5: VIN, Connector_PinSocket_2.54mm:PinSocket_1x02_P2.54mm_Vertical, F.Cu at (6.51, -50.0)
- added J6: VOUT, TerminalBlock_Phoenix:TerminalBlock_Phoenix_MKDS-1,5-2-5.08_1x02_P5.08mm_Horizontal, F.Cu at (-10.3, -38.8)
- added JP1: LED_EN, Jumper:SolderJumper-2_P1.3mm_Open_TrianglePad1.0x1.5mm, F.Cu at (6.36, -38.3)
- added JS1: JOY_PSP, DPX_CONTROL:JOYSTICK-PSP1000_mars, F.Cu at (-37.1, -80.5)
- added JS2: JOY_PSP, DPX_CONTROL:JOYSTICK-PSP1000_mars, F.Cu at (-16.0, -80.5)
- added JS3: JOY_PSP, DPX_CONTROL:JOYSTICK-PSP1000_mars, F.Cu at (5.09, -80.5)
- added JS4: JOY_PSP, DPX_CONTROL:JOYSTICK-PSP1000_mars, F.Cu at (26.2, -80.5)
- added LED1: XL_WS2812B_4020, DPX_LED:LED_WS2812_4020, F.Cu at (-35.2, -66.5)
- added LED10: GREEN, DPX_LED:LED_0805_2012Metric_Pad1.15x1.40mm_HandSolder, F.Cu at (1.81, -60.1)
- added LED11: YELLO, DPX_LED:LED_0805_2012Metric_Pad1.15x1.40mm_HandSolder, F.Cu at (1.81, -57.1)
- added LED2: XL_WS2812B_4020, DPX_LED:LED_WS2812_4020, F.Cu at (-35.2, -63.5)
- added LED3: XL_WS2812B_4020, DPX_LED:LED_WS2812_4020, F.Cu at (-35.2, -60.5)
- added LED4: XL_WS2812B_4020, DPX_LED:LED_WS2812_4020, F.Cu at (-35.2, -57.5)
- added LED5: XL_WS2812B_4020, DPX_LED:LED_WS2812_4020, F.Cu at (-35.2, -54.5)
- added LED6: XL_WS2812B_4020, DPX_LED:LED_WS2812_4020, F.Cu at (-35.2, -51.5)
- added LED7: XL_WS2812B_4020, DPX_LED:LED_WS2812_4020, F.Cu at (-35.2, -48.5)
- added LED8: XL_WS2812B_4020, DPX_LED:LED_WS2812_4020, F.Cu at (-35.2, -45.5)
- added LED9: RED, DPX_LED:LED_0805_2012Metric_Pad1.15x1.40mm_HandSolder, F.Cu at (1.81, -63.2)
- added R1: 680R, Resistor_SMD:R_0603_1608Metric_Pad0.98x0.95mm_HandSolder, F.Cu at (-2.96, -53.8)
- added R2: 680R, Resistor_SMD:R_0603_1608Metric_Pad0.98x0.95mm_HandSolder, F.Cu at (-2.96, -51.3)
- added R3: 680R, Resistor_SMD:R_0603_1608Metric_Pad0.98x0.95mm_HandSolder, F.Cu at (-2.96, -48.8)
- added R4: 1k, Resistor_SMD:R_0805_2012Metric_Pad1.20x1.40mm_HandSolder, F.Cu at (-25.2, -48.2)
- added R5: 10k, Resistor_SMD:R_0805_2012Metric_Pad1.20x1.40mm_HandSolder, F.Cu at (-25.2, -45.3)
- added R6: 1k, Resistor_SMD:R_0805_2012Metric_Pad1.20x1.40mm_HandSolder, F.Cu at (-25.2, -42.3)
- added R7: 10k, Resistor_SMD:R_0805_2012Metric_Pad1.20x1.40mm_HandSolder, F.Cu at (-25.2, -39.4)
- added R8: 10k, Resistor_SMD:R_0805_2012Metric_Pad1.20x1.40mm_HandSolder, F.Cu at (-25.2, -36.4)
- added R9: 10k, Resistor_SMD:R_0805_2012Metric_Pad1.20x1.40mm_HandSolder, F.Cu at (-25.2, -33.5)
- added SW1: SW_DIP_x03, DPX_CONTROL:SP-03P, F.Cu at (8.73, -62.2)
- added SYM1: Logo_Open_Hardware_Small, DPX_LIBRARY:OSHW-LogoNT_7.3x6mm_Silk, F.Cu at (6.98, -42.3)
- added U10: R-785.0-0.5, Converter_DCDC:Converter_DCDC_RECOM_R-78E-0.5_THT, F.Cu at (-9.67, -60.5)
- added U11: CH224K, Package_SO:SSOP-10-1EP_3.9x4.9mm_P1mm_EP2.1x3.3mm_ThermalVias, F.Cu at (27.3, -64.3)
- added U5: TC118S, DPX_IC:SOP-8_3.76x4.96mm_P1.27mm, F.Cu at (98.5, -24.7)
- added U6: TC118S, DPX_IC:SOP-8_3.76x4.96mm_P1.27mm, F.Cu at (76.1, 187.6)
- added U7: TC118S, DPX_IC:SOP-8_3.76x4.96mm_P1.27mm, F.Cu at (98.5, -18.0)
- added U8: TC118S, DPX_IC:SOP-8_3.76x4.96mm_P1.27mm, F.Cu at (98.5, -11.4)
- added U9: Teensy4.1, teensy:Teensy41, F.Cu at (47.0, -15.1)
- added USB1: HRO-TYPE-C-31-M-12, DPX_USB:HRO-TYPE-C-31-M-12-Assembly, F.Cu at (17.8, -58.7)
- J1: value Conn_01x08_Pin -> motor.1; footprint Connector_PinHeader_2.54mm:PinHeader_1x08_P2.54mm_Vertical -> Connector_JST:JST_PH_B2B-PH-SM4-TB_1x02-1MP_P2.00mm_Vertical
- J2: value Conn_01x08_Pin -> motor.2; footprint Connector_PinHeader_2.54mm:PinHeader_1x08_P2.54mm_Vertical -> Connector_JST:JST_PH_B2B-PH-SM4-TB_1x02-1MP_P2.00mm_Vertical
- U1, U2, U3, U4: value ~ -> SM100BN-B10K; footprint DPX_CONTROL:Fader_apai_SC1009M -> DPX_CONTROL:Fader_terwin_SM100BN-B10K--L82T1H5
- moved J1 160.1 mm to (-43.0, -62.5), turned to 0 degrees
- moved J2 134.4 mm to (-43.0, -52.9), turned to 0 degrees
- moved U1 4.31 mm to (58.4, 109.0)
- moved U2 2.53 mm to (76.0, 109.0)
- moved U4 1.19 mm to (111.2, 109.0)
- moved U3 0.81 mm to (93.6, 109.0)
Connections:
- net VCC renamed +3.3V
- J1 pad 1: /P1 -> motor.1-NEG
- J1 pad 2: /T1 -> motor.1-POS
- J2 pad 1: /M1_A -> motor.2-NEG
- J2 pad 2: /M1_B -> motor.2-POS
- U1 pad 2: /P1 -> wiper_1
- U1 pad 4: GND -> unconnected-(U1B-Touch-Pad4)
- U1 pad 5: /M1_A -> motor.1-POS
- U1 pad 6: /M1_B -> motor.1-NEG
- U2 pad 2: /P2 -> wiper_2
- U2 pad 4: GND -> unconnected-(U2B-Touch-Pad4)
- U2 pad 5: /M2_A -> motor.2-POS
- U2 pad 6: /M2_B -> motor.2-NEG
- U3 pad 2: /P3 -> wiper_3
- U3 pad 4: GND -> unconnected-(U3B-Touch-Pad4)
- U3 pad 5: /M3_A -> motor.3-POS
- U3 pad 6: /M3_B -> unconnected-(U3C---Pad6)
- U4 pad 2: /P4 -> wiper_4
- U4 pad 4: GND -> unconnected-(U4B-Touch-Pad4)
- U4 pad 5: /M4_A -> motor.4-POS
- U4 pad 6: /M4_B -> motor.4-NEG
Routing:
- net /T1: track 165.5 -> 0.00 mm
- net /M4_B: track 156.7 -> 0.00 mm
- net /M4_A: track 156.3 -> 0.00 mm
- net /T2: track 149.3 -> 0.00 mm
- net /T4: track 146.9 -> 0.00 mm
- net /M3_B: track 143.3 -> 0.00 mm
- net /M3_A: track 143.3 -> 0.00 mm
- net /T3: track 142.5 -> 0.00 mm
- net /M2_B: track 141.3 -> 0.00 mm
- net /M2_A: track 141.0 -> 0.00 mm
- net /M1_B: track 138.3 -> 0.00 mm
- net /M1_A: track 138.3 -> 0.00 mm
- net /P1: track 47.9 -> 0.00 mm
- net /P2: track 30.6 -> 0.00 mm
- net /P3: track 17.7 -> 0.00 mm
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- added copper zone on In1.Cu, net (none)
- removed copper zone on In1.Cu, net +3.3V
Other:
- board text removed: "1.A"
- board text removed: "1.B"
- board text removed: "1.P"
- board text removed: "1.T"
- board text removed: "2.A"
- board text removed: "2.B"
- board text removed: "2.P"
- board text removed: "2.T"
- board text removed: "3.A"
- board text removed: "3.B"
- board text removed: "3.P"
- board text removed: "3.T"
- board text removed: "4.A"
- board text removed: "4.B"
- board text removed: "4.P"
- board text removed: "4.T"

Commit message: first release
** big reorganize
++ version 1.0 of FADED4_LYFE based on v1.8 of FADE4
++ lots of fader related spec sheets.
--remove backup files and other erratta
Parts:
- removed D1: MBRA130LT3G, Diode_SMD:D_SMA
- removed D2: VBUS, DPX_LED:LED_0805_2012Metric_Pad1.15x1.40mm_HandSolder
- removed FB1: 220h 110mHz, DPX_USB:FERRITE_0603
- removed J5: VIN, Connector_PinSocket_2.54mm:PinSocket_1x02_P2.54mm_Vertical
- removed J6: VOUT, TerminalBlock_Phoenix:TerminalBlock_Phoenix_MKDS-1,5-2-5.08_1x02_P5.08mm_Horizontal
- removed JP1: LED_EN, Jumper:SolderJumper-2_P1.3mm_Open_TrianglePad1.0x1.5mm
- removed JS1, JS2, JS3, JS4: JOY_PSP, DPX_CONTROL:JOYSTICK-PSP1000_mars
- removed LED1, LED2, LED3, LED4, LED5, LED6, LED7, LED8: XL_WS2812B_4020, DPX_LED:LED_WS2812_4020
- removed R4, R6: 1k, Resistor_SMD:R_0805_2012Metric_Pad1.20x1.40mm_HandSolder
- removed R5, R7, R8, R9: 10k, Resistor_SMD:R_0805_2012Metric_Pad1.20x1.40mm_HandSolder
- removed U1, U2, U3, U4: SM100BN-B10K, DPX_CONTROL:Fader_terwin_SM100BN-B10K--L82T1H5
- removed USB1: HRO-TYPE-C-31-M-12, DPX_USB:HRO-TYPE-C-31-M-12-Assembly
- added C20: 100 NF, Capacitor_SMD:C_0603_1608Metric_Pad1.08x0.95mm_HandSolder, F.Cu at (284.6, 156.6)
- added C21: 100 nF, Capacitor_SMD:C_0805_2012Metric_Pad1.18x1.45mm_HandSolder, F.Cu at (352.2, 143.2)
- added DC1: DC-005-5A-2.0-SMT, EasyEda-Automatic:DC-IN-TH_DC-005-5A-2.0-SMT, F.Cu at (368.0, 165.8)
- added R10: 680R, Resistor_SMD:R_0603_1608Metric_Pad0.98x0.95mm_HandSolder, F.Cu at (367.7, 138.3)
- added RJ1: J1B1211CCD, EasyEda-Automatic:RJ45-TH_J1B1211CCD, F.Cu at (363.0, 147.6)
- added SW2: TS-1187A-B-A-B, EasyEda-Automatic:SW-SMD_4P-L5.1-W5.1-P3.70-LS6.5-TL_H1.5, F.Cu at (340.8, 173.8)
- added U12: NML0505SC, DPX_IC:NML0505SC, F.Cu at (336.4, 142.0)
- added U13: ~, DPX_CONTROL:Fader_behringerx32_b10k_100mm, B.Cu at (315.2, 172.2)
- added U14: ~, DPX_CONTROL:Fader_behringerx32_b10k_100mm, B.Cu at (289.8, 172.3)
- added kibuzzard-67C38035: G***, kibuzzard-67C38035, F.Cu at (366.3, 231.9)
- added kibuzzard-67C38035: G***, kibuzzard-67C38035, B.Cu at (366.2, 232.0)
- added kibuzzard-67C38056: G***, kibuzzard-67C38056, F.Cu at (341.1, 232.2)
- added kibuzzard-67C38056: G***, kibuzzard-67C38056, B.Cu at (341.0, 232.2)
- added kibuzzard-67C38062: G***, kibuzzard-67C38062, F.Cu at (315.7, 232.1)
- added kibuzzard-67C38062: G***, kibuzzard-67C38062, B.Cu at (315.6, 232.2)
- added kibuzzard-67C38072: G***, kibuzzard-67C38072, F.Cu at (289.9, 232.3)
- added kibuzzard-67C38072: G***, kibuzzard-67C38072, B.Cu at (289.9, 232.2)
- added kibuzzard-67C38A3C: G***, kibuzzard-67C38A3C, F.Cu at (329.0, 222.3)
- added kibuzzard-67C38B05: G***, kibuzzard-67C38B05, B.Cu at (329.0, 222.2)
- added kibuzzard-67C3BB4B: G***, kibuzzard-67C3BB4B, B.Cu at (352.5, 178.4)
- C1, C10, C4, C7: footprint Capacitor_SMD:C_0805_2012Metric_Pad1.18x1.45mm_HandSolder -> Capacitor_SMD:C_1206_3216Metric_Pad1.33x1.80mm_HandSolder
- C11, C12, C2, C3, C5, C6, C8, C9: value 100 uF -> 100 NF
- C13: value .1 uF -> 100 nF
- C14, C16: value 10uF -> 100 NF; footprint Capacitor_SMD:CP_Elec_5x5.8 -> Capacitor_SMD:C_0603_1608Metric_Pad1.08x0.95mm_HandSolder
- C15: value 10uF -> 100 NF; footprint Capacitor_SMD:C_0805_2012Metric_Pad1.18x1.45mm_HandSolder -> Capacitor_SMD:C_0603_1608Metric_Pad1.08x0.95mm_HandSolder
- C17, C18, C19: value 1 uF -> 100 NF
- H1, H2, H3, H4: footprint MountingHole:MountingHole_2.2mm_M2_ISO7380_Pad_TopBottom -> MountingHole:MountingHole_4.3mm_M4_ISO14580
- J1, J2, J3, J4: footprint Connector_JST:JST_PH_B2B-PH-SM4-TB_1x02-1MP_P2.00mm_Vertical -> EasyEda-Automatic:CONN-SMD_PH2.0-1X2PW
- SW1: value SW_DIP_x03 -> TS-1187A-B-A-B; footprint DPX_CONTROL:SP-03P -> EasyEda-Automatic:SW-SMD_4P-L5.1-W5.1-P3.70-LS6.5-TL_H1.5
- U10: value R-785.0-0.5 -> ~; footprint Converter_DCDC:Converter_DCDC_RECOM_R-78E-0.5_THT -> DPX_CONTROL:Fader_behringerx32_b10k_100mm; moved to B.Cu
- U11: value CH224K -> ~; footprint Package_SO:SSOP-10-1EP_3.9x4.9mm_P1mm_EP2.1x3.3mm_ThermalVias -> DPX_CONTROL:Fader_behringerx32_b10k_100mm; moved to B.Cu
- U5, U6, U7, U8: footprint DPX_IC:SOP-8_3.76x4.96mm_P1.27mm -> EasyEda-Automatic:SOP-8_L4.9-W3.9-P1.27-LS6.0-BL
- U9: footprint teensy:Teensy41 -> DPX_IC:Teensy41_less_pins
- moved H4 472.9 mm to (353.3, 226.8)
- moved J1 445.7 mm to (365.8, 115.2)
- moved U10 441.9 mm to (366.0, 172.2), turned to -90 degrees
- moved R3 440.6 mm to (374.7, 178.2), turned to -90 degrees
- moved LED11 438.8 mm to (374.6, 174.5), turned to 90 degrees
- moved C7 437.0 mm to (370.3, 125.6)
- moved H3 436.1 mm to (302.6, 226.8)
- moved LED9 433.4 mm to (374.6, 158.0), turned to -90 degrees
- moved C13 427.7 mm to (357.1, 137.5), turned to 180 degrees
- moved SYM1 422.3 mm to (328.4, 231.6)
- moved H2 422.2 mm to (353.4, 116.3)
- moved LED10 421.8 mm to (374.6, 137.1), turned to -90 degrees
- moved R2 420.3 mm to (374.7, 133.2), turned to 90 degrees
- moved R1 419.6 mm to (359.3, 157.8), turned to 180 degrees
- moved C3 419.6 mm to (370.3, 119.7), turned to 90 degrees
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Connections:
- C1 pad 1: +3.3V -> +5v-DIRTY
- C10 pad 1: +3.3V -> +5v-DIRTY
- C14 pad 1: Net-(D1-K) -> +3.3V
- C15 pad 1: +5v-vIN -> +3.3V
- C16 pad 1: +5v-vIN -> +3.3V
- C17 pad 1: +5v-vIN -> wiper_1
- C18 pad 1: +5v-vIN -> wiper_2
- C19 pad 1: VDD -> wiper_3
- C4 pad 1: +3.3V -> +5v-DIRTY
- C7 pad 1: +3.3V -> +5v-DIRTY
- J1 pad 1: motor.1-NEG -> motor.1-POS
- J1 pad 2: motor.1-POS -> motor.1-NEG
- J2 pad 1: motor.2-NEG -> motor.2-POS
- J2 pad 2: motor.2-POS -> motor.2-NEG
- J3 pad 1: motor.3-NEG -> motor.3-POS
- J3 pad 2: motor.3-POS -> motor.3-NEG
- J4 pad 1: motor.4-NEG -> motor.4-POS
- J4 pad 2: motor.4-POS -> motor.4-NEG
- LED10 pad 1: GND -> Net-(LED10-A)
- LED10 pad 2: Net-(LED10-A) -> GND
- LED11 pad 1: GND -> Net-(LED11-A)
- LED11 pad 2: Net-(LED11-A) -> GND
- LED9 pad 1: GND -> Net-(LED9-A)
- LED9 pad 2: Net-(LED9-A) -> GND
- R1 pad 2: Net-(JP1-A) -> 13_SCK
- R2 pad 2: +5V -> +3.3V
- SW1 pad 1: GND -> BUTTON1
- SW1 pad 2: GND -> unconnected-(SW1-B-Pad2)
- SW1 pad 3: GND -> unconnected-(SW1-C-Pad3)
- SW1 pad 4: CFG3 -> GND
- U10 pad 1: Net-(D1-K) -> GND
- U10 pad 2: GND -> wiper_1
- U10 pad 3: +5v-vIN -> +3.3V
- U11 pad 1: VDD -> GND
- U11 pad 2: CFG2 -> wiper_2
- U11 pad 3: CFG3 -> +3.3V
- U11 pad 4: D+ -> wiper_2
- U11 pad 7: CC1 -> (no net)
- U5 pad 4: +3.3V -> +5v-DIRTY
- U6 pad 4: +3.3V -> +5v-DIRTY
- U7 pad 4: +3.3V -> +5v-DIRTY
- U8 pad 4: +3.3V -> +5v-DIRTY
- U9 pad 10: mc4.U -> unconnected-(U9-8_TX2_IN1-Pad10)
- U9 pad 11: mc4.D -> unconnected-(U9-9_OUT1C-Pad11)
- U9 pad 15: +3.3V -> unconnected-(U9-3V3-Pad15)
- U9 pad 16: joy4.x -> unconnected-(U9-24_A10_TX6_SCL2-Pad16)
- U9 pad 17: joy4.y -> unconnected-(U9-25_A11_RX6_SDA2-Pad17)
- U9 pad 2: unconnected-(U9-0_RX1_CRX2_CS1-Pad2) -> mc1.U
- U9 pad 21: touch_1 -> unconnected-(U9-29_TX7-Pad21)
- U9 pad 22: touch_2 -> unconnected-(U9-30_CRX3-Pad22)
- U9 pad 23: touch_3 -> unconnected-(U9-31_CTX3-Pad23)
- U9 pad 24: touch_4 -> LED6
- U9 pad 25: unconnected-(U9-33_MCLK2-Pad25) -> BUTTON2
- U9 pad 3: unconnected-(U9-1_TX1_CTX2_MISO1-Pad3) -> mc1.D
- U9 pad 33: unconnected-(U9-41_A17-Pad33) -> BUTTON1
- U9 pad 35: unconnected-(U9-13_SCK_LED-Pad35) -> 13_SCK
- U9 pad 36: wiper_4 -> unconnected-(U9-14_A0_TX3_SPDIF_OUT-Pad36)
- U9 pad 37: wiper_3 -> unconnected-(U9-15_A1_RX3_SPDIF_IN-Pad37)
- U9 pad 38: wiper_2 -> unconnected-(U9-16_A2_RX4_SCL1-Pad38)
- U9 pad 39: wiper_1 -> unconnected-(U9-17_A3_TX4_SDA1-Pad39)
- U9 pad 4: mc1.U -> mc2.U
- U9 pad 40: joy3.y -> unconnected-(U9-18_A4_SDA-Pad40)
- U9 pad 41: joy3.x -> unconnected-(U9-19_A5_SCL-Pad41)
- U9 pad 42: joy2.y -> wiper_4
- U9 pad 43: joy2.x -> wiper_3
- U9 pad 44: joy1.y -> wiper_2
- U9 pad 45: joy1.x -> wiper_1
- U9 pad 5: mc1.D -> mc2.D
- U9 pad 6: mc2.U -> mc3.U
- U9 pad 60: Net-(U9-R+) -> R+
- U9 pad 61: Net-(RJ1-LLED+) -> LLED+
- U9 pad 62: Net-(U9-T-) -> T-
- U9 pad 63: Net-(U9-T+) -> T+
- U9 pad 64: Net-(C13-Pad1) -> GND
- U9 pad 65: Net-(U9-R-) -> R-
- U9 pad 7: mc2.D -> mc3.D
- U9 pad 8: mc3.U -> mc4.U
- U9 pad 9: mc3.D -> mc4.D
Routing:
- net wiper_1: track 0.00 -> 172.1 mm
- net +5v-DIRTY: track 0.00 -> 169.2 mm, vias 0 -> 4
- net +3.3V: track 0.00 -> 161.5 mm, vias 0 -> 4
- net wiper_2: track 0.00 -> 152.6 mm
- net wiper_3: track 0.00 -> 133.9 mm
- net wiper_4: track 0.00 -> 118.0 mm
- net mc1.U: track 0.00 -> 115.3 mm, vias 0 -> 1
- net mc1.D: track 0.00 -> 108.2 mm, vias 0 -> 1
- net +5v-CLEAN: track 0.00 -> 96.5 mm
- net mc2.U: track 0.00 -> 83.0 mm, vias 0 -> 1
- net LLED+: track 0.00 -> 77.6 mm, vias 0 -> 1
- net mc2.D: track 0.00 -> 76.6 mm, vias 0 -> 1
- net T-: track 0.00 -> 70.9 mm
- net T+: track 0.00 -> 70.7 mm
- net R+: track 0.00 -> 62.7 mm
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- added copper zone on In1.Cu, net GND
- removed copper zone on In1.Cu, net (none)
- removed copper zone on In2.Cu, net GND
Other:
- board size 185.1 x 165 mm -> 96.5 x 132.7 mm
- board text added: "${COMPANY} - ${ISSUE_DATE}"
- board text added: "${TITLE}"
- board text added: "${TITLE} // ${REVISION} - ${ISSUE_DATE}"
- board text added: "DHCP"
- board text added: "STATIC"
- board text added: "U5"
- board text added: "U6"
- board text added: "U7"
- board text added: "U8"
- board text added: "hey! heres an absurdly large box to write something in <3"
- board text removed: "1"
- board text removed: "2"
- board text removed: "3"
- board text removed: "4"
- board text removed: "dpx_faded"
- board text removed: "dpx_faded.fbd // v1d0 - 11.8.24"
