File: hardware/src/dpx_faded/dpx_faded.kicad_pcb (KiCad board)
At the start: 4 copper layers, 96.5 x 132.7 mm, 75 parts, among them J1 motor.1, J2 motor.2, J3 motor.3, J4 motor.4, SW1 TS-1187A-B-A-B, SW2 TS-1187A-B-A-B, U1 CH224K, U12 NML0505SC, U5 TC118S, U6 TC118S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

Commit message: firmware and hardware fixes
-------//FIRMWARE
** changed static/reset ip to 10.0 values (see reset.ino&WebServerApply.Ino) 10.0.10.130 & sending to 10.0.10.120
++ added maxpatch to test midi / motor functionality
++ 3mf for the enclosure
------//HARDWARE
** corrected some LED pinout shiz, other stuff.
Parts:
- added kibuzzard-67D0F279: G***, kibuzzard-67D0F279, B.Cu at (328.1, 191.1)
- moved R9 53.1 mm to (360.5, 191.3), turned to 180 degrees
- moved U1 50.6 mm to (360.5, 185.5), turned to 90 degrees
- moved R13 49.8 mm to (359.9, 168.0), turned to 90 degrees
- moved R11 49.6 mm to (359.9, 164.2), turned to 90 degrees
- moved R12 42.9 mm to (369.5, 157.2), turned to 180 degrees
- moved LED1 42.1 mm to (373.8, 191.5), turned to 180 degrees
- moved LED2 42.0 mm to (373.5, 157.2), turned to 180 degrees
- moved LED9 39.8 mm to (373.7, 174.0), turned to 180 degrees
- moved LED11 39.8 mm to (373.7, 177.6), turned to 180 degrees
- moved USB1 34.4 mm to (375.9, 197.7), turned to 90 degrees
- moved USB2 25.5 mm to (375.9, 185.7), turned to 90 degrees
- moved kibuzzard-67CFB29D 1.44 mm to (302.4, 190.9)
- moved kibuzzard-67C3BB4B 1.39 mm to (353.2, 177.2)
- moved LED10 1.32 mm to (373.4, 137.6), turned to 0 degrees
- renumbered SW2 to SW1, SW1 to SW2
Connections:
- LED1 pad 1: Net-(LED1-A) -> PG
- LED1 pad 2: PG -> Net-(LED1-C)
- LED10 pad 1: Net-(LED10-A) -> GND
- LED10 pad 2: GND -> Net-(LED10-C)
- LED11 pad 1: Net-(LED11-A) -> GND
- LED11 pad 2: GND -> Net-(LED11-A)
- LED2 pad 1: Net-(LED2-A) -> GND
- LED2 pad 2: GND -> Net-(LED2-C)
- LED9 pad 1: Net-(LED9-A) -> GND
- LED9 pad 2: GND -> Net-(LED9-C)
- R11 pad 1: Net-(LED9-A) -> Net-(LED9-C)
- R12 pad 1: Net-(LED2-A) -> Net-(LED2-C)
- R2 pad 1: Net-(LED10-A) -> Net-(LED10-C)
- R9 pad 1: Net-(LED1-A) -> Net-(LED1-C)
Routing:
- net LED6: track 51.8 -> 24.3 mm
- net Net-(LED9-A): track 14.7 -> 0.00 mm
- net 13_SCK: track 52.5 -> 56.9 mm
- net Net-(LED10-C): track 0.00 -> 3.60 mm
- net GND: track 43.0 -> 41.1 mm, vias 22 -> 21
- net Net-(LED11-A): track 1.78 -> 0.00 mm

Commit message: refresh base files and push some pcb stuff
Parts:
- added J5: Conn_01x02_Pin, DPX_DUMP:1X02, F.Cu at (372.1, 205.7)
- added JP1: Jumper_3_Bridged12, Jumper:SolderJumper-3_P1.3mm_Bridged12_RoundedPad1.0x1.5mm_NumberLabels, F.Cu at (358.1, 208.8)
- moved FB1 62.7 mm to (366.0, 202.2), turned to 90 degrees
- moved R4 58.3 mm to (359.8, 188.2), turned to 180 degrees
- moved R5 57.5 mm to (360.9, 192.1), turned to -90 degrees
- moved FB2 56.1 mm to (365.7, 190.0), turned to 90 degrees
- moved C22 56.1 mm to (358.8, 192.2), turned to 90 degrees
- moved R9 12.3 mm to (358.2, 203.4), turned to 90 degrees
- moved U1 12.3 mm to (360.1, 197.8)
Connections:
- U12 pad 2: +5v-DIRTY -> Net-(JP1-C)
- U9 pad 66: unconnected-(U9-D--Pad66) -> D-2
- U9 pad 67: unconnected-(U9-D+-Pad67) -> D+2
- USB2 pad 5: D- -> D-2
- USB2 pad 6: D+ -> D+2
- USB2 pad 7: D- -> D-2
- USB2 pad 8: D+ -> D+2
