File: hardware/src/dpx_faded/dpx_faded.kicad_sch (KiCad schematic)
At the start: 6 parts, among them J1 Conn_01x08_Pin, J2 Conn_01x08_Pin

Commit message: so much source and so much datasheet
lots of fader drama
gonna fork the design and reduce featureset, add x32 faders due to availa
basically make a FADE_4 clone first because well - that whole thing has turned into the mystery project
Parts:
- removed J1, J2: Conn_01x08_Pin, Connector_PinHeader_2.54mm:PinHeader_1x08_P2.54mm_Vertical, symbol Connector:Conn_01x08_Pin
- removed U1, U2, U3, U4: ~, DPX_CONTROL:Fader_apai_SC1009M, symbol DPX_CONTROL:Touch_Fader_Motorized
- added C1, C10, C4, C7: 4.7 uF, Capacitor_SMD:C_0805_2012Metric_Pad1.18x1.45mm_HandSolder, symbol Device:C_Small
- added C11, C12, C2, C3, C5, C6, C8, C9: 100 uF, Capacitor_SMD:C_0603_1608Metric_Pad1.08x0.95mm_HandSolder, symbol Device:C_Small
- added C13: .1 uF, Capacitor_SMD:C_0805_2012Metric_Pad1.18x1.45mm_HandSolder, symbol Device:C_Small
- added C14, C16: 10uF, Capacitor_SMD:CP_Elec_5x5.8, symbol Device:C_Polarized_Small
- added C15: 10uF, Capacitor_SMD:C_0805_2012Metric_Pad1.18x1.45mm_HandSolder, symbol DPX_POOP:C_Small
- added C17, C18, C19: 1 uF, Capacitor_SMD:C_0603_1608Metric_Pad1.08x0.95mm_HandSolder, symbol DPX_POOP:C_Small
- added D1: MBRA130LT3G, Diode_SMD:D_SMA, symbol Device:D_Schottky
- added D2: VBUS, DPX_LED:LED_0805_2012Metric_Pad1.15x1.40mm_HandSolder, symbol Device:LED
- added FB1: 220h 110mHz, DPX_USB:FERRITE_0603, symbol Device:FerriteBead_Small
- added H1, H2, H3, H4: MountingHole_Pad_MP, MountingHole:MountingHole_2.2mm_M2_ISO7380_Pad_TopBottom, symbol Mechanical:MountingHole_Pad_MP
- added J1: motor.1, Connector_JST:JST_PH_B2B-PH-SM4-TB_1x02-1MP_P2.00mm_Vertical, symbol Connector:Conn_01x02_Pin
- added J2: motor.2, Connector_JST:JST_PH_B2B-PH-SM4-TB_1x02-1MP_P2.00mm_Vertical, symbol Connector:Conn_01x02_Pin
- added J3: motor.3, Connector_JST:JST_PH_B2B-PH-SM4-TB_1x02-1MP_P2.00mm_Vertical, symbol Connector:Conn_01x02_Pin
- added J4: motor.4, Connector_JST:JST_PH_B2B-PH-SM4-TB_1x02-1MP_P2.00mm_Vertical, symbol Connector:Conn_01x02_Pin
- added J5: VIN, Connector_PinSocket_2.54mm:PinSocket_1x02_P2.54mm_Vertical, symbol Connector:Conn_01x02_Socket
- added J6: VOUT, TerminalBlock_Phoenix:TerminalBlock_Phoenix_MKDS-1,5-2-5.08_1x02_P5.08mm_Horizontal, symbol Connector:Conn_01x02_Socket
- added JP1: LED_EN, Jumper:SolderJumper-2_P1.3mm_Open_TrianglePad1.0x1.5mm, symbol Jumper:Jumper_2_Small_Open
- added JS1, JS2, JS3, JS4: JOY_PSP, DPX_CONTROL:JOYSTICK-PSP1000_mars, symbol DPX_CONTROL:JOYSTICK-PSP1K
- added LED1, LED2, LED3, LED4, LED5, LED6, LED7, LED8: XL_WS2812B_4020, DPX_LED:LED_WS2812_4020, symbol DPX_LED:XL-WS2812B_4020
- added LED10: GREEN, DPX_LED:LED_0805_2012Metric_Pad1.15x1.40mm_HandSolder, symbol DPX_LED:LED
- added LED11: YELLO, DPX_LED:LED_0805_2012Metric_Pad1.15x1.40mm_HandSolder, symbol DPX_LED:LED
- added LED9: RED, DPX_LED:LED_0805_2012Metric_Pad1.15x1.40mm_HandSolder, symbol DPX_LED:LED
- added R1, R2, R3: 680R, Resistor_SMD:R_0603_1608Metric_Pad0.98x0.95mm_HandSolder, symbol DPX_POOP:R
- added R10: 680R, symbol DPX_EXPORT_DUMP1:R_Small
- added R4, R6: 1k, Resistor_SMD:R_0805_2012Metric_Pad1.20x1.40mm_HandSolder, symbol Device:R
- added R5, R7, R8, R9: 10k, Resistor_SMD:R_0805_2012Metric_Pad1.20x1.40mm_HandSolder, symbol Device:R
- added RJ1: J1B1211CCD, EasyEDA:RJ45-TH_J1B1211CCD, symbol EasyEDA-AutoImport:J1B1211CCD
- added SW1: SW_DIP_x03, DPX_CONTROL:SP-03P, symbol Switch:SW_DIP_x03
- added SYM1: Logo_Open_Hardware_Small, DPX_LIBRARY:OSHW-LogoNT_7.3x6mm_Silk, symbol Graphic:Logo_Open_Hardware_Small
- added U1, U2, U3, U4: SM100BN-B10K, DPX_CONTROL:Fader_terwin_SM100BN-B10K--L82T1H5, symbol DPX_CONTROL:Touch_Fader_terwin_SM100BN-B10K--L82T1H5
- added U10: R-785.0-0.5, Converter_DCDC:Converter_DCDC_RECOM_R-78E-0.5_THT, symbol Regulator_Switching:R-785.0-0.5
- added U11: CH224K, Package_SO:SSOP-10-1EP_3.9x4.9mm_P1mm_EP2.1x3.3mm_ThermalVias, symbol DPX_IC:CH224K
- added U12: NML0505SC, symbol DPX_IC:NML0505SC
- added U5, U6, U7, U8: TC118S, DPX_IC:SOP-8_3.76x4.96mm_P1.27mm, symbol DPX_IC:TC118S
- added U9: Teensy4.1, teensy:Teensy41, symbol teensy:Teensy4.1
- added USB1: HRO-TYPE-C-31-M-12, DPX_USB:HRO-TYPE-C-31-M-12-Assembly, symbol DPX_USB:HRO-TYPE-C-31-M-12
Connections:
- net GND: now also C1.2, C10.2, C14.2, C15.2, C16.2, C17.2, C18.2, C19.2, C4.2, C7.2, FB1.2, J5.1 (Pin_1), J6.2 (Pin_2), JS1.2 (GND), JS2.2 (GND), JS3.2 (GND), JS4.2 (GND), LED1.4 (VSS), LED10.1 (C), LED11.1 (C), LED2.4 (VSS), LED3.4 (VSS), LED4.4 (VSS), LED5.4 (VSS), LED6.4 (VSS), LED7.4 (VSS), LED8.4 (VSS), LED9.1 (C), SW1.1, SW1.2, SW1.3, U1.1 (VCC), U10.2 (GND), U11.11 (GND), U11.9 (CFG1), U12.1 (VIN-), U12.3 (VOUT-), U2.1 (VCC), U3.1 (VCC), U4.1 (VCC), U5.6 (AGND), U5.7 (PGND), U6.6 (AGND), U6.7 (PGND), U7.6 (AGND), U7.7 (PGND), U8.6 (AGND), U8.7 (PGND), U9.1 (GND), U9.34 (GND), U9.47 (GND), USB1.1 (GND), USB1.12 (GND)
- new net: LED2.3 (DOUT), LED3.1 (DIN)
- new net: LED3.3 (DOUT), LED4.1 (DIN)
- new net: C14.1, D1.1 (K), U10.1 (IN)
- new net: R5.2, U11.8 (VBUS)
- new net: LED9.2 (A), R1.1
- new net: JP1.1 (A), R1.2
- new net: LED6.3 (DOUT), LED7.1 (DIN)
- new net: LED7.3 (DOUT), LED8.1 (DIN)
- new net: D2.2 (A), R6.1
- new net: RJ1.1, U9.63 (T+)
- new net: RJ1.10 (LLED+), U9.61 (LED)
- new net: C13.1, RJ1.2, RJ1.5, U9.64 (GND)
- new net: RJ1.3, U9.62 (T-)
- new net: RJ1.4, U9.60 (R+)
- new net: RJ1.6, U9.65 (R-)
- new net: C13.2, RJ1.8
- new net: LED11.2 (A), R3.1
- new net: LED1.3 (DOUT), LED2.1 (DIN)
- new net: FB1.1, USB1.13 (SHIELD)
- new net: LED10.2 (A), R2.1
- new net: LED5.3 (DOUT), LED6.1 (DIN)
- new net +3.3V: C1.1, C10.1, C4.1, C7.1, JS1.4 (VCC), JS2.4 (VCC), JS3.4 (VCC), JS4.4 (VCC), LED1.2 (VDD), LED2.2 (VDD), LED3.2 (VDD), LED4.2 (VDD), LED5.2 (VDD), LED6.2 (VDD), LED7.2 (VDD), LED8.2 (VDD), U1.3 (GND), U2.3 (GND), U3.3 (GND), U4.3 (GND), U5.4 (VDD), U6.4 (VDD), U7.4 (VDD), U8.4 (VDD), U9.15 (3V3), U9.46 (3V3)
- new net +5V: R2.2
- new net +5v-CLEAN: R10.2, U12.4 (VOUT+), U9.48 (VIN)
- new net +5v-vIN: C15.1, C16.1, C17.1, C18.1, U10.3 (OUT), U12.2 (VIN+)
- new net 13_SCK: JP1.2 (B)
- new net CC1: U11.7 (CC1), USB1.4 (CC1)
- new net CC2: U11.6 (CC2), USB1.10 (CC2)
- new net CFG1: R7.2, SW1.6
- new net CFG2: R8.2, SW1.5, U11.2 (CFG2)
- new net CFG3: R9.2, SW1.4, U11.3 (CFG3)
- new net D+: U11.4 (D+), USB1.6 (DP1), USB1.8 (DP2)
- new net D-: U11.5 (D-), USB1.5 (DN2), USB1.7 (DN1)
- new net GND2: RJ1.11 (RLED-), RJ1.13 (GND), RJ1.14 (GND), RJ1.9 (LLED-)
- new net LED6: R3.2
- new net LLED+: R10.1, RJ1.12 (RLED+)
- new net PG: D2.1 (K), U11.10 (PG)
- new net VBUS: J6.1 (Pin_1), R4.1, R5.1, USB1.11 (VBUS), USB1.2 (VBUS)
- new net VDD: C19.1, R4.2, R6.2, R7.1, R8.1, R9.1, U11.1 (VDD)
- new net VLED: D1.2 (A), J5.2 (Pin_2)
- new net joy1.x: JS1.1 (X), U9.45 (23_A9_CRX1_MCLK1)
- new net joy1.y: JS1.3 (Y), U9.44 (22_A8_CTX1)
- new net joy2.x: JS2.1 (X), U9.43 (21_A7_RX5_BCLK1)
- new net joy2.y: JS2.3 (Y), U9.42 (20_A6_TX5_LRCLK1)
- new net joy3.x: JS3.1 (X), U9.41 (19_A5_SCL)
- new net joy3.y: JS3.3 (Y), U9.40 (18_A4_SDA)
- new net joy4.x: JS4.1 (X), U9.16 (24_A10_TX6_SCL2)
- new net joy4.y: JS4.3 (Y), U9.17 (25_A11_RX6_SDA2)
- new net led_group_2: LED4.3 (DOUT), LED5.1 (DIN)
- new net led_in: LED1.1 (DIN)
- new net mc1.D: U5.3 (IN-B), U9.5 (3_LRCLK2)
- new net mc1.U: U5.2 (IN-A), U9.4 (2_OUT2)
- new net mc2.D: U6.3 (IN-B), U9.7 (5_IN2)
- new net mc2.U: U6.2 (IN-A), U9.6 (4_BCLK2)
- new net mc3.D: U7.3 (IN-B), U9.9 (7_RX2_OUT1A)
- new net mc3.U: U7.2 (IN-A), U9.8 (6_OUT1D)
- new net mc4.D: U8.3 (IN-B), U9.11 (9_OUT1C)
- new net mc4.U: U8.2 (IN-A), U9.10 (8_TX2_IN1)
- new net motor.1-NEG: C2.2, C3.2, J1.1 (Pin_1), U1.6 (-), U5.5 (OUTB)
- new net motor.1-POS: C2.1, C3.1, J1.2 (Pin_2), U1.5 (+), U5.8 (OUTA)
- new net motor.2-NEG: C5.2, C6.2, J2.1 (Pin_1), U2.6 (-), U6.5 (OUTB)
- new net motor.2-POS: C5.1, C6.1, J2.2 (Pin_2), U2.5 (+), U6.8 (OUTA)
- new net motor.3-NEG: C8.2, C9.2, J3.1 (Pin_1), U7.5 (OUTB)
- new net motor.3-POS: C8.1, C9.1, J3.2 (Pin_2), U3.5 (+), U7.8 (OUTA)
- new net motor.4-NEG: C11.2, C12.2, J4.1 (Pin_1), U4.6 (-), U8.5 (OUTB)
- new net motor.4-POS: C11.1, C12.1, J4.2 (Pin_2), U4.5 (+), U8.8 (OUTA)
- new net touch_1: U1.0 (Touch), U9.21 (29_TX7)
- new net touch_2: U2.0 (Touch), U9.22 (30_CRX3)
- new net touch_3: U3.0 (Touch), U9.23 (31_CTX3)
- new net touch_4: U4.0 (Touch), U9.24 (32_OUT1B)
- new net wiper_1: U1.2 (Wiper), U9.39 (17_A3_TX4_SDA1)
- new net wiper_2: U2.2 (Wiper), U9.38 (16_A2_RX4_SCL1)
- new net wiper_3: U3.2 (Wiper), U9.37 (15_A1_RX3_SPDIF_IN)
- new net wiper_4: U4.2 (Wiper), U9.36 (14_A0_TX3_SPDIF_OUT)
Other:
- note added: "dubpixel"

Commit message: first release
** big reorganize
++ version 1.0 of FADED4_LYFE based on v1.8 of FADE4
++ lots of fader related spec sheets.
--remove backup files and other erratta
Parts:
- removed C14, C16: 10uF, Capacitor_SMD:CP_Elec_5x5.8, symbol Device:C_Polarized_Small
- removed C15: 10uF, Capacitor_SMD:C_0805_2012Metric_Pad1.18x1.45mm_HandSolder, symbol DPX_POOP:C_Small
- removed C17, C18, C19: 1 uF, Capacitor_SMD:C_0603_1608Metric_Pad1.08x0.95mm_HandSolder, symbol DPX_POOP:C_Small
- removed D1: MBRA130LT3G, Diode_SMD:D_SMA, symbol Device:D_Schottky
- removed D2: VBUS, DPX_LED:LED_0805_2012Metric_Pad1.15x1.40mm_HandSolder, symbol Device:LED
- removed FB1: 220h 110mHz, DPX_USB:FERRITE_0603, symbol Device:FerriteBead_Small
- removed J5: VIN, Connector_PinSocket_2.54mm:PinSocket_1x02_P2.54mm_Vertical, symbol Connector:Conn_01x02_Socket
- removed J6: VOUT, TerminalBlock_Phoenix:TerminalBlock_Phoenix_MKDS-1,5-2-5.08_1x02_P5.08mm_Horizontal, symbol Connector:Conn_01x02_Socket
- removed JP1: LED_EN, Jumper:SolderJumper-2_P1.3mm_Open_TrianglePad1.0x1.5mm, symbol Jumper:Jumper_2_Small_Open
- removed JS1, JS2, JS3, JS4: JOY_PSP, DPX_CONTROL:JOYSTICK-PSP1000_mars, symbol DPX_CONTROL:JOYSTICK-PSP1K
- removed LED1, LED2, LED3, LED4, LED5, LED6, LED7, LED8: XL_WS2812B_4020, DPX_LED:LED_WS2812_4020, symbol DPX_LED:XL-WS2812B_4020
- removed R4, R6: 1k, Resistor_SMD:R_0805_2012Metric_Pad1.20x1.40mm_HandSolder, symbol Device:R
- removed R5, R7, R8, R9: 10k, Resistor_SMD:R_0805_2012Metric_Pad1.20x1.40mm_HandSolder, symbol Device:R
- removed SW1: SW_DIP_x03, DPX_CONTROL:SP-03P, symbol Switch:SW_DIP_x03
- removed U1, U2, U3, U4: SM100BN-B10K, DPX_CONTROL:Fader_terwin_SM100BN-B10K--L82T1H5, symbol DPX_CONTROL:Touch_Fader_terwin_SM100BN-B10K--L82T1H5
- removed U10: R-785.0-0.5, Converter_DCDC:Converter_DCDC_RECOM_R-78E-0.5_THT, symbol Regulator_Switching:R-785.0-0.5
- removed U11: CH224K, Package_SO:SSOP-10-1EP_3.9x4.9mm_P1mm_EP2.1x3.3mm_ThermalVias, symbol DPX_IC:CH224K
- removed USB1: HRO-TYPE-C-31-M-12, DPX_USB:HRO-TYPE-C-31-M-12-Assembly, symbol DPX_USB:HRO-TYPE-C-31-M-12
- added C14, C15, C16, C17, C18, C19, C20: 100 NF, Capacitor_SMD:C_0603_1608Metric_Pad1.08x0.95mm_HandSolder, symbol Device:C_Small
- added C21: 100 nF, Capacitor_SMD:C_0805_2012Metric_Pad1.18x1.45mm_HandSolder, symbol Device:C_Small
- added DC1: DC-005-5A-2.0-SMT, EasyEda-Automatic:DC-IN-TH_DC-005-5A-2.0-SMT, symbol EasyEDA-AutoImport:DC-005-5A-2.0-SMT
- added SW1, SW2: TS-1187A-B-A-B, EasyEda-Automatic:SW-SMD_4P-L5.1-W5.1-P3.70-LS6.5-TL_H1.5, symbol EasyEDA-AutoImport:TS-1187A-B-A-B
- added U10, U11, U13, U14: ~, DPX_CONTROL:Fader_behringerx32_b10k_100mm, symbol DPX_CONTROL:Behringer_X32_Fader_Motorized
- C1, C10, C4, C7: footprint Capacitor_SMD:C_0805_2012Metric_Pad1.18x1.45mm_HandSolder -> Capacitor_SMD:C_1206_3216Metric_Pad1.33x1.80mm_HandSolder; LCSC (none) -> C29823
- C11, C12, C2, C3, C5, C6, C8, C9: value 100 uF -> 100 NF; LCSC (none) -> C14663
- C13: value .1 uF -> 100 nF; LCSC (none) -> C14663
- H1, H2, H3, H4: footprint MountingHole:MountingHole_2.2mm_M2_ISO7380_Pad_TopBottom -> MountingHole:MountingHole_4.3mm_M4_ISO14580
- J1, J2, J3, J4: footprint Connector_JST:JST_PH_B2B-PH-SM4-TB_1x02-1MP_P2.00mm_Vertical -> EasyEda-Automatic:CONN-SMD_PH2.0-1X2PW; LCSC (none) -> C64658
- R10: footprint (none) -> Resistor_SMD:R_0603_1608Metric_Pad0.98x0.95mm_HandSolder
- RJ1: footprint EasyEDA:RJ45-TH_J1B1211CCD -> EasyEda-Automatic:RJ45-TH_J1B1211CCD; LCSC (none) -> C910371
- U12: footprint (none) -> DPX_IC:NML0505SC
- U5, U6, U7, U8: footprint DPX_IC:SOP-8_3.76x4.96mm_P1.27mm -> EasyEda-Automatic:SOP-8_L4.9-W3.9-P1.27-LS6.0-BL
- U9: footprint teensy:Teensy41 -> DPX_IC:Teensy41_less_pins
Connections:
- net +5V is gone; now on net +3.3V: R2.2
- net GND2 is gone; now on net GND: RJ1.11 (RLED-), RJ1.13 (GND), RJ1.14 (GND), RJ1.9 (LLED-)
- net joy1.x is gone; now on net wiper_1: U9.45 (23_A9_CRX1_MCLK1)
- net joy1.y is gone; now on net wiper_2: U9.44 (22_A8_CTX1)
- net joy2.x is gone; now on net wiper_3: U9.43 (21_A7_RX5_BCLK1)
- net joy2.y is gone; now on net wiper_4: U9.42 (20_A6_TX5_LRCLK1)
- net touch_4 is gone; now on net LED6: U9.24 (32_OUT1B)
- net +3.3V: now also C14.1, C15.1, C16.1, U10.3 (GND), U11.3 (GND), U13.3 (GND), U14.3 (GND); no longer C1.1, C10.1, C4.1, C7.1, U5.4 (VDD), U6.4 (VDD), U7.4 (VDD), U8.4 (VDD), U9.15 (3V3)
- net 13_SCK: now also R1.2, U9.35 (13_SCK_LED)
- net GND: now also LED10.2 (C), LED11.2 (C), LED9.2 (C), U9.64 (GND), C14.2, C15.2, C16.2, C17.2, C18.2, C19.2, C20.2, C21.2, DC1.2, SW1.4 (D), SW2.4 (D), U10.1 (VCC), U11.1 (VCC), U13.1 (VCC), U14.1 (VCC); no longer LED10.1 (C), LED11.1 (C), LED9.1 (C)
- net LLED+: now also RJ1.10 (LLED+), U9.61 (LED); no longer R10.1, RJ1.12 (RLED+)
- net mc1.D: now also U9.3 (1_TX1_CTX2_MISO1); no longer U9.5 (3_LRCLK2)
- net mc1.U: now also U9.2 (0_RX1_CRX2_CS1); no longer U9.4 (2_OUT2)
- net mc2.D: now also U9.5 (3_LRCLK2); no longer U9.7 (5_IN2)
- net mc2.U: now also U9.4 (2_OUT2); no longer U9.6 (4_BCLK2)
- net mc3.D: now also U9.7 (5_IN2); no longer U9.9 (7_RX2_OUT1A)
- net mc3.U: now also U9.6 (4_BCLK2); no longer U9.8 (6_OUT1D)
- net mc4.D: now also U9.9 (7_RX2_OUT1A); no longer U9.11 (9_OUT1C)
- net mc4.U: now also U9.8 (6_OUT1D); no longer U9.10 (8_TX2_IN1)
- net motor.1-NEG: now also J1.2 (Pin_2), U10.6 (-); no longer J1.1 (Pin_1)
- net motor.1-POS: now also J1.1 (Pin_1), U10.5 (+); no longer J1.2 (Pin_2)
- net motor.2-NEG: now also J2.2 (Pin_2), U11.6 (-); no longer J2.1 (Pin_1)
- net motor.2-POS: now also J2.1 (Pin_1), U11.5 (+); no longer J2.2 (Pin_2)
- net motor.3-NEG: now also J3.2 (Pin_2), U13.6 (-); no longer J3.1 (Pin_1)
- net motor.3-POS: now also J3.1 (Pin_1), U13.5 (+); no longer J3.2 (Pin_2)
- net motor.4-NEG: now also J4.2 (Pin_2), U14.6 (-); no longer J4.1 (Pin_1)
- net motor.4-POS: now also J4.1 (Pin_1), U14.5 (+); no longer J4.2 (Pin_2)
- net wiper_1: now also C17.1, U10.2 (Wiper), U10.4; no longer U9.39 (17_A3_TX4_SDA1)
- net wiper_2: now also C18.1, U11.2 (Wiper), U11.4; no longer U9.38 (16_A2_RX4_SCL1)
- net wiper_3: now also C19.1, U13.2 (Wiper), U13.4; no longer U9.37 (15_A1_RX3_SPDIF_IN)
- net wiper_4: now also C20.1, U14.2 (Wiper), U14.4; no longer U9.36 (14_A0_TX3_SPDIF_OUT)
- net at R1.1: now also LED9.1 (A); no longer LED9.2 (A)
- net T+: now reaches RJ1.1, U9.63 (T+)
- net at C13.1, RJ1.2, RJ1.5: no longer U9.64 (GND)
- net T-: now reaches RJ1.3, U9.62 (T-)
- net R+: now reaches RJ1.4, U9.60 (R+)
- net R-: now reaches RJ1.6, U9.65 (R-)
- net at C13.2, RJ1.8: now also C21.1
- net at R3.1: now also LED11.1 (A); no longer LED11.2 (A)
- net BUTTON2: now reaches U9.25 (33_MCLK2)
- net BUTTON2: now also SW2.2 (B)
- net BUTTON1: now reaches U9.33 (41_A17)
- net BUTTON1: now also SW1.1 (A)
- net at R2.1: now also LED10.1 (A); no longer LED10.2 (A)
- net +5v-vIN renamed +5v-DIRTY
- net +5v-DIRTY: now also C1.1, C10.1, C4.1, C7.1, U5.4 (VDD), U6.4 (VDD), U7.4 (VDD), U8.4 (VDD), DC1.1
- net joy3.x: no longer names the net of U9.41 (19_A5_SCL)
- net joy3.y: no longer names the net of U9.40 (18_A4_SDA)
- net joy4.x: no longer names the net of U9.16 (24_A10_TX6_SCL2)
- net joy4.y: no longer names the net of U9.17 (25_A11_RX6_SDA2)
- net touch_1: no longer names the net of U9.21 (29_TX7)
- net touch_2: no longer names the net of U9.22 (30_CRX3)
- net touch_3: no longer names the net of U9.23 (31_CTX3)
- new net RLED+: R10.1, RJ1.12 (RLED+)
Other:
- note added: "DHCP"
- note added: "Fader fader1(A9, 0); Fader fader2(A8, 1); Fader fader3(A7, 2); Fader fader4(A6, 3); Fader fader5(A5, 4); Fader fader6(A4, 5); Fader fader7(A3, 6); Fader fader8(A2, 7);"
- note added: "STATIC"
- note added: "static byte PINS_1_A[8] = {0, 2, 4, 6, 8, 10, 24, 28}; static byte PINS_1_B[8] = {1, 3, 5, 7, 9, 12, 25, 29};"
- title: (none) -> dpx_faded_4_lyfe
- moved on the sheet: C1, C10, C11, C12, C2, C3, C4, C5, C6, C7, C8, C9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

Commit message: schematic stuff
** cleanup schematic
++ 74HC4051 mux
++ 4x joysticks
Parts:
- added JS1, JS2, JS3, JS4: JOY_PSP, DPX_CONTROL:JOYSTICK-PSP1000_mars, symbol DPX_CONTROL:JOYSTICK-PSP1K
- added U1: 74HC4051, Package_SO:TSSOP-16_4.4x5mm_P0.65mm, symbol 74xx:74HC4051
Connections:
- net +3.3V: now also JS1.4 (VCC), JS2.4 (VCC), JS3.4 (VCC), JS4.4 (VCC), U1.16 (VCC)
- net +5v-CLEAN: no longer R10.2, U12.4 (VOUT+)
- net GND: now also JS1.2 (GND), JS2.2 (GND), JS3.2 (GND), JS4.2 (GND), U1.8 (GND)
- net MUX_1.3: now reaches U9.26 (34_RX8)
- net MUX_1.3: now also U1.9 (S2)
- net MUX_1.2: now reaches U9.27 (35_TX8)
- net MUX_1.2: now also U1.10 (S1)
- net MUX_1.1: now reaches U9.28 (36_CS)
- net MUX_1.1: now also U1.11 (S0)
- net analog_mux1: now reaches U9.36 (14_A0_TX3_SPDIF_OUT)
- net analog_mux1: now also U1.3 (A)
- net wiper_8: now reaches U9.38 (16_A2_RX4_SCL1)
- net wiper_7: now reaches U9.39 (17_A3_TX4_SDA1)
- net wiper_6: now reaches U9.40 (18_A4_SDA)
- net wiper_5: now reaches U9.41 (19_A5_SCL)
- new net: R10.2, U12.4 (VOUT+)
- new net j1.x: JS1.1 (X), U1.13 (A0)
- new net j1.y: JS1.3 (Y), U1.14 (A1)
- new net j2.x: JS2.1 (X), U1.15 (A2)
- new net j2.y: JS2.3 (Y), U1.12 (A3)
- new net j3.x: JS3.1 (X), U1.1 (A4)
- new net j3.y: JS3.3 (Y), U1.5 (A5)
- new net j4.x: JS4.1 (X), U1.2 (A6)
- new net j4.y: JS4.3 (Y), U1.4 (A7)
Other:
- moved on the sheet: C1, C10, C11, C12, C13, C14, C15, C16, C17, C18, C19, C2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

Commit message: joysticks... but going back to the main branch to make some easier changes
Parts:
- added J5, J6: Conn_01x03_Socket, Connector_JST:JST_PH_S3B-PH-SM4-TB_1x03-1MP_P2.00mm_Horizontal, symbol Connector:Conn_01x03_Socket
- added J7, J8: Conn_01x03_Pin, Connector_JST:JST_PH_S3B-PH-SM4-TB_1x03-1MP_P2.00mm_Horizontal, symbol Connector:Conn_01x03_Pin
Connections:
- net +3.3V: now also J6.1 (Pin_1), J7.1 (Pin_1)
- net +5v-CLEAN: now also R10.2, U12.4 (VOUT+)
- net GND: now also U1.6 (~{E}), J6.3 (Pin_3), J7.3 (Pin_3)
- net MUX_1.1: now also J5.1 (Pin_1), J8.1 (Pin_1)
- net MUX_1.2: now also J5.2 (Pin_2), J8.2 (Pin_2)
- net MUX_1.3: now also J5.3 (Pin_3), J8.3 (Pin_3)
- net analog_mux1: now also J6.2 (Pin_2), J7.2 (Pin_2)
Other:
- note added: "no pin 7 on symbol (this is the moutn hole)"
- note added: "no pins 3/4 - these are the mounting tabs on the jst connector"
- moved on the sheet: U1
