File: hardware/src/dpx_faded/dpx_faded.kicad_sch (KiCad schematic)
At the start: 51 parts, among them J1 motor.1, J2 motor.2, J3 motor.3, J4 motor.4, SW1 TS-1187A-B-A-B, SW2 TS-1187A-B-A-B, U12 NML0505SC, U5 TC118S, U6 TC118S, U7 TC118S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

Commit message: post v0.5.0 fixes--->(v0.6.0)
-----//HARDWARE
++ CH244 PD controller rough in
++ update PCB
++ add pdf for a fader

-----//FIRMWARE
++ add maxpatch to test faders
Parts:
- removed R1, R3: 680R, Resistor_SMD:R_0603_1608Metric_Pad0.98x0.95mm_HandSolder, symbol DPX_POOP:R
- added C22: 1 uF, Capacitor_SMD:C_0603_1608Metric_Pad1.08x0.95mm_HandSolder, symbol DPX_POOP:C_Small
- added FB1, FB2: 220h 110mHz, DPX_USB:FERRITE_0603, symbol Device:FerriteBead_Small
- added LED1: RED, LED_SMD:LED_0603_1608Metric_Pad1.05x0.95mm_HandSolder, symbol DPX_LED:LED
- added LED2: GREEN, DPX_LED:LED_0805_2012Metric_Pad1.15x1.40mm_HandSolder, symbol DPX_LED:LED
- added R11: 75R, Resistor_SMD:R_0603_1608Metric_Pad0.98x0.95mm_HandSolder, symbol DPX_POOP:R
- added R12, R13, R9: 120R, Resistor_SMD:R_0603_1608Metric_Pad0.98x0.95mm_HandSolder, symbol DPX_POOP:R
- added R4: 1k, Resistor_SMD:R_0805_2012Metric_Pad1.20x1.40mm_HandSolder, symbol Device:R
- added R5: 10k, Resistor_SMD:R_0805_2012Metric_Pad1.20x1.40mm_HandSolder, symbol Device:R
- added U1: CH224K, Package_SO:SSOP-10-1EP_3.9x4.9mm_P1mm_EP2.1x3.3mm_ThermalVias, symbol DPX_IC:CH224K
- added USB1, USB2: HRO-TYPE-C-31-M-12, DPX_USB:HRO-TYPE-C-31-M-12-Assembly, symbol DPX_USB:HRO-TYPE-C-31-M-12
- LED10: value GREEN -> YELLO; LCPART C2297 -> C2296; LCSC C2297 -> C2296
- LED11: value YELLO -> WHITE; LCPART C2296 -> C34499; LCSC C2296 -> C34499
- LED9: LCPART C2296 -> C84256
- R2: value 680R -> 65R; LCPART C23228 -> (none); LCSC C23228 -> (none)
Connections:
- net 13_SCK: now also R11.2
- net GND: now also C22.2, FB1.2, FB2.2, LED2.2 (C), U1.11 (GND), USB1.1 (GND), USB1.12 (GND), USB2.1 (GND), USB2.12 (GND)
- net LED6: now also R13.2
- net at LED9.1 (A): now also R11.1
- net at LED11.1 (A): now also R13.1
- net VBUS_uC: now reaches U9.49 (VUSB)
- net VBUS_uC: now also USB2.11 (VBUS), USB2.2 (VBUS)
- new net: LED2.1 (A), R12.1
- new net: R5.2, U1.8 (VBUS)
- new net: FB1.1, USB1.13 (SHIELD)
- new net: LED1.1 (A), R9.1
- new net: FB2.1, USB2.13 (SHIELD)
- new net +5V: R12.2
- new net CC1: U1.7 (CC1), USB1.4 (CC1), USB2.4 (CC1)
- new net CC2: U1.6 (CC2), USB1.10 (CC2), USB2.10 (CC2)
- new net CFG2: U1.2 (CFG2)
- new net CFG3: U1.3 (CFG3)
- new net D+: U1.4 (D+), USB1.6 (DP1), USB1.8 (DP2), USB2.6 (DP1), USB2.8 (DP2)
- new net D-: U1.5 (D-), USB1.5 (DN2), USB1.7 (DN1), USB2.5 (DN2), USB2.7 (DN1)
- new net PG: LED1.2 (C), U1.10 (PG)
- new net VBUS: R4.1, R5.1, USB1.11 (VBUS), USB1.2 (VBUS)
- new net VDD: C22.1, R4.2, R9.2, U1.1 (VDD), U1.9 (CFG1)
Other:
- note added: "VF RED = 1.6 MIN /2.0/ 2.6 MAX - 25mA@ 3v3 72R 0.045 watt"
- note added: "VF WHITE = 2.6 MIN / -- / 3.2 MAX - 5mA@ 3v3 140R 0.0035 watt 120ohm..."
- note added: "VF YELLO = 2.0 MIN /2--/ 2.2 MAX - 20mA@ 3v3 65R 0.026 watt"
- note added: "VFGREEN = 2.8 /MAX 2.9 (LETS DO 2.7 at 5v supply) 20 MA 120OHM"
- moved on the sheet: LED10, R2

Commit message: firmware and hardware fixes
-------//FIRMWARE
** changed static/reset ip to 10.0 values (see reset.ino&WebServerApply.Ino) 10.0.10.130 & sending to 10.0.10.120
++ added maxpatch to test midi / motor functionality
++ 3mf for the enclosure
------//HARDWARE
** corrected some LED pinout shiz, other stuff.
Parts:
- SW1: renamed from SW2; footprint EasyEda-Automatic:SW-SMD_4P-L5.1-W5.1-P3.70-LS6.5-TL_H1.5 -> EasyEDA:SW-SMD_4P-L5.1-W5.1-P3.70-LS6.5-TL_H1.5
- SW2: renamed from SW1; footprint EasyEda-Automatic:SW-SMD_4P-L5.1-W5.1-P3.70-LS6.5-TL_H1.5 -> EasyEDA:SW-SMD_4P-L5.1-W5.1-P3.70-LS6.5-TL_H1.5
Connections:
- net GND: now also LED10.1 (C), LED11.1 (C), LED2.1 (C), LED9.1 (C); no longer LED10.2 (C), LED11.2 (C), LED2.2 (C), LED9.2 (C)
- net PG: now also LED1.1 (C); no longer LED1.2 (C)
- net at R12.1: now also LED2.2 (A); no longer LED2.1 (A)
- net at R13.1: now also LED11.2 (A); no longer LED11.1 (A)
- net at R9.1: now also LED1.2 (A); no longer LED1.1 (A)
- net at R11.1: now also LED9.2 (A); no longer LED9.1 (A)
- net at R2.1: now also LED10.2 (A); no longer LED10.1 (A)
Changed lines of the file:
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@@
 			)
 		)
-		(property "Description" ""
+		(property "Description" "Resistor"
 			(at 52.07 60.96 0)
 			(effects
@@
 		(dnp no)
 		(fields_autoplaced yes)
-		(property "Reference" "SW1"
+		(property "Reference" "SW2"
 			(at 238.76 78.74 0)
 			(effects
@@
 			)
 		)
-		(property "Footprint" "EasyEda-Automatic:SW-SMD_4P-L5.1-W5.1-P3.70-LS6.5-TL_H1.5"
+		(property "Footprint" "EasyEDA:SW-SMD_4P-L5.1-W5.1-P3.70-LS6.5-TL_H1.5"
 			(at 238.76 99.06 0)
 			(effects
@@
 			(project ""
 				(path "/730caac5-d131-4da1-a76c-40d992583383"
-					(reference "SW1")
+					(reference "SW2")
 					(unit 1)
 				)
@@
 		(dnp no)
 		(fields_autoplaced yes)
-		(property "Reference" "SW2"
+		(property "Reference" "SW1"
 			(at 260.35 78.74 0)
 			(effects
@@
 			)
 		)
-		(property "Footprint" "EasyEda-Automatic:SW-SMD_4P-L5.1-W5.1-P3.70-LS6.5-TL_H1.5"
+		(property "Footprint" "EasyEDA:SW-SMD_4P-L5.1-W5.1-P3.70-LS6.5-TL_H1.5"
 			(at 260.35 99.06 0)
 			(effects
@@
 			(project "dpx_faded"
 				(path "/730caac5-d131-4da1-a76c-40d992583383"
-					(reference "SW2")
+					(reference "SW1")
 					(unit 1)
 				)
@@
 			)
 		)
+		(property "Sim.Enable" "0"
+			(at 307.34 261.62 0)
+			(effects
+				(font
+					(size 1.27 1.27)
+				)
+				(hide yes)
+			)
+		)
 		(instances
 			(project "dpx_faded"
@@
 			)
 		)
-		(property "Description" ""
+		(property "Description" "Resistor"
 			(at 62.23 67.31 0)
 			(effects

Commit message: refresh base files and push some pcb stuff
Parts:
- added J5: Conn_01x02_Pin, DPX_DUMP:1X02, symbol Connector:Conn_01x02_Pin
- added JP1: Jumper_3_Bridged12, Jumper:SolderJumper-3_P1.3mm_Bridged12_RoundedPad1.0x1.5mm_NumberLabels, symbol Jumper:Jumper_3_Bridged12
Connections:
- net +5v-DIRTY: now also JP1.2 (C)
- net D+: no longer USB2.6 (DP1), USB2.8 (DP2)
- net D-: no longer USB2.5 (DN2), USB2.7 (DN1)
- net GND: now also J5.2 (Pin_2)
- net VBUS: now also JP1.1 (A)
- net D-2: now reaches U9.66 (D-)
- net D-2: now also USB2.5 (DN2), USB2.7 (DN1)
- net D+2: now reaches U9.67 (D+)
- net D+2: now also USB2.6 (DP1), USB2.8 (DP2)
- new net: J5.1 (Pin_1), JP1.3 (B)
